File: board-game-timer_hardware/board-game-timer_hardware.kicad_pcb (KiCad board)
At the start: 4 copper layers, 100 x 65 mm, 45 parts, among them J1 USB_B_Micro, J2 boot0_jumper, J3 BIG_SWITCH_HEADER, J4 JTAG_HEADER, Q1 BC847C,215, SW1 SW_RST, SW2 EC11E15244G1, U1 STM32F030F4Px, U2 AMS1117-3.3, U3 TM1637, U4 FJ5462AH, Y1 16MHz

Commit message: Made changes to make board 10mm less wide
Parts:
- BZ1: value Buzzer -> Fengming YS-MBZ12085C05R42
- moved C7 11.8 mm to (102.6, 65.5)
- moved D1 11.8 mm to (110.0, 73.9)
- moved R1 11.8 mm to (106.8, 74.0)
- moved U2 11.8 mm to (108.7, 66.4)
- moved C6 11.1 mm to (115.7, 63.2)
- moved J1 11.1 mm to (121.7, 62.9)
- moved J4 10.5 mm to (117.0, 29.8)
- moved H2 10.0 mm to (120.0, 20.0)
- moved H4 10.0 mm to (120.0, 75.0)
Routing:
- net SW_CLK: track 60.3 -> 49.9 mm, vias 0 -> 1
- net SW_DIO: track 59.0 -> 48.8 mm
- net RST: track 77.6 -> 68.6 mm, vias 2 -> 0
- net GND: track 67.5 -> 66.3 mm, vias 46 -> 44
- net /RED-: track 1.90 -> 3.20 mm, vias 0 -> 1
- net Net-(J1-VBUS): track 6.63 -> 7.28 mm
Other:
- board size 100 x 65 mm -> 90 x 65 mm
- board text added: "Made by Krzysztof github.com/Krisss99/game-board-timer v1.1"
- board text removed: "Made by Krzysztof Cajler github.com/Krisss99/game-board-timer v1.1"
